File: pcb/pcb.kicad_sch (KiCad schematic)
At the start: 0 parts

Commit message: added all the keys to the schematic
yay
Parts:
- added D1, D10, D11, D12, D13, D14, D15, D16, D17, D18, D19, D2, D20, D21, D22, D23, D24, D25, D26, D27, D28, D29, D3, D30, D31, D32, D33, D34, D35, D36, D37, D38, D39, D4, D40, D41, D42, D43, D44, D45, D46, D47, D48, D49, D5, D50, D51, D52, D53, D54, D55, D56, D57, D58, D59, D6, D60, D61, D62, D63, D64, D65, D66, D67, D68, D69, D7, D70, D71, D72, D73, D74, D75, D76, D77, D78, D79, D8, D80, D9: D, symbol Device:D
- added SW1, SW10, SW11, SW12, SW13, SW14, SW15, SW16, SW17, SW18, SW19, SW2, SW20, SW21, SW22, SW23, SW24, SW25, SW26, SW27, SW28, SW29, SW3, SW30, SW31, SW32, SW33, SW34, SW35, SW36, SW37, SW38, SW39, SW4, SW40, SW41, SW42, SW43, SW44, SW45, SW46, SW47, SW48, SW49, SW5, SW50, SW51, SW52, SW53, SW54, SW55, SW56, SW57, SW58, SW59, SW6, SW60, SW61, SW62, SW63, SW64, SW65, SW66, SW67, SW68, SW69, SW7, SW70, SW71, SW72, SW73, SW74, SW75, SW76, SW77, SW78, SW79, SW8, SW80, SW9: SW_Push, symbol Switch:SW_Push
- added U1: RP2350_80QFN, RP2350_80QFN_minimal:RP2350-QFN-80-1EP_10x10_P0.4mm_EP3.4x3.4mm_ThermalVias, symbol MCU_RaspberryPi_RP2350:RP2350_80QFN
Connections:
- new net: D18.2 (A), SW18.2
- new net: D3.2 (A), SW3.2
- new net: D78.2 (A), SW78.2
- new net: D80.2 (A), SW80.2
- new net: D12.2 (A), SW12.2
- new net: D61.2 (A), SW61.2
- new net: D66.2 (A), SW66.2
- new net: D68.2 (A), SW68.2
- new net: D53.2 (A), SW53.2
- new net: D26.2 (A), SW26.2
- new net: D17.2 (A), SW17.2
- new net: D71.2 (A), SW71.2
- new net: D42.2 (A), SW42.2
- new net: D56.2 (A), SW56.2
- new net: D25.2 (A), SW25.2
- new net: D37.2 (A), SW37.2
- new net: D50.2 (A), SW50.2
- new net: D48.2 (A), SW48.2
- new net: D75.2 (A), SW75.2
- new net: D77.2 (A), SW77.2
- new net: D52.2 (A), SW52.2
- new net: D10.2 (A), SW10.2
- new net: D16.2 (A), SW16.2
- new net: D62.2 (A), SW62.2
- new net: D8.2 (A), SW8.2
- new net: D72.2 (A), SW72.2
- new net: D9.2 (A), SW9.2
- new net: D19.2 (A), SW19.2
- new net: D7.2 (A), SW7.2
- new net: D29.2 (A), SW29.2
- new net: D36.2 (A), SW36.2
- new net: D4.2 (A), SW4.2
- new net: D13.2 (A), SW13.2
- new net: D55.2 (A), SW55.2
- new net: D40.2 (A), SW40.2
- new net: D23.2 (A), SW23.2
- new net: D43.2 (A), SW43.2
- new net: D54.2 (A), SW54.2
- new net: D57.2 (A), SW57.2
- new net: D60.2 (A), SW60.2
- new net: D58.2 (A), SW58.2
- new net: D76.2 (A), SW76.2
- new net: D38.2 (A), SW38.2
- new net: D33.2 (A), SW33.2
- new net: D11.2 (A), SW11.2
- new net: D15.2 (A), SW15.2
- new net: D21.2 (A), SW21.2
- new net: D74.2 (A), SW74.2
- new net: D45.2 (A), SW45.2
- new net: D6.2 (A), SW6.2
- new net: D47.2 (A), SW47.2
- new net: D64.2 (A), SW64.2
- new net: D67.2 (A), SW67.2
- new net: D24.2 (A), SW24.2
- new net: D69.2 (A), SW69.2
- new net: D30.2 (A), SW30.2
- new net: D59.2 (A), SW59.2
- new net: D32.2 (A), SW32.2
- new net: D34.2 (A), SW34.2
- new net: D27.2 (A), SW27.2
- new net: D70.2 (A), SW70.2
- new net: D28.2 (A), SW28.2
- new net: D35.2 (A), SW35.2
- new net: D51.2 (A), SW51.2
- new net: D63.2 (A), SW63.2
- new net: D49.2 (A), SW49.2
- new net: D65.2 (A), SW65.2
- new net: D31.2 (A), SW31.2
- new net: D79.2 (A), SW79.2
- new net: D5.2 (A), SW5.2
- new net: D22.2 (A), SW22.2
- new net: D20.2 (A), SW20.2
- new net: D41.2 (A), SW41.2
- new net: D14.2 (A), SW14.2
- new net: D1.2 (A), SW1.2
- new net: D2.2 (A), SW2.2
- new net: D39.2 (A), SW39.2
- new net: D46.2 (A), SW46.2
- new net: D44.2 (A), SW44.2
- new net: D73.2 (A), SW73.2
